File: Gamepad PCB/Gamepad PCB.kicad_sch (KiCad schematic)
At the start: 119 parts, among them J1 USB_C_16P, J2 XH2.54, J3 XH2.54, J4 XH2.54, J5 XH2.54, J6 XH2.54, J7 XH2.54, M1 Vibration Motor, Q1 Si2301, Q2 SS8050, Q3 IRF4905, Q4 SS8050, Q5 2N2222, Q6 2N2222, Q7 Si2300, Q8 Si2300, SW1 SW_Push, SW10 Ctrl button, SW11 Config switch, SW12 Corner switch, SW13 Adj button, SW14 Ctrl button, SW15 Config switch, SW16 Corner switch, SW17 Adj button, SW18 Ctrl button, SW19 Config switch, SW2 RST Button, SW3 Boot Button, SW4 Corner button, SW5 Adj button, SW6 Ctrl button, SW7 Config switch, SW8 Corner button, SW9 Adj button, U1 AMS1117-3.3, U10 CP2102, U11 ADS1015IDGS, U12 74HC4051, U13 74HC165D, U2 LC709203FQH-01TWG, U3 USBLC6-2SC6, U4 NRF24L01 PA + LNA, U5 AMS1117-3.3, U6 ESP32-S3-WROOM1, U7 TP4056, U8 DW01A, U9 8205

Commit message: add imgs
Other:
- company: (none) -> PCM Industries
- title: (none) -> Multipurpose ESP32 Gamepad
Changed lines of the file:
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@@
 	(generator_version "9.0")
 	(paper "A4")
+	(title_block
+		(title "Multipurpose ESP32 Gamepad")
+		(date "2025-07-30")
+		(rev "v03")
+		(company "PCM Industries")
+		(comment 1 "Author: Pacman Ng")
+		(comment 2 "Manufacturer: JLCPCB")
+	)
 	(rectangle
 		(start 113.03 64.77)

Commit message: fix entire pcb
Parts:
- added D10, D11, D12, D13, D14, D15, D16, D17, D18, D19, D20, D21, D6, D7, D8, D9: 1N4007, Diode_SMD:D_SOD-123, symbol Device:D_Small
- U7: footprint Package_SO:SOP-8-1EP_4.57x4.57mm_P1.27mm_EP4.57x4.45mm -> Package_SO:HTSOP-8-1EP_3.9x4.9mm_P1.27mm_EP2.4x3.2mm_ThermalVias
Connections:
- net GPIO0 is gone; now on net IO0: Q4.3 (C)
- net +3.3V_Perip: now also J7.7 (Pin_7); no longer J7.2 (Pin_2)
- net +BATT: now also Q3.2; no longer Q3.3, R4.1
- net CLK: now also J7.6 (Pin_6); no longer J7.3 (Pin_3)
- net GND: now also J7.8 (Pin_8); no longer J7.1 (Pin_1)
- net IO17: now also J7.1 (Pin_1); no longer J7.5 (Pin_5)
- net IO18: now also J7.2 (Pin_2); no longer J7.6 (Pin_6)
- net IO19: now also J7.3 (Pin_3); no longer J7.7 (Pin_7)
- net IO20: now also J7.4 (Pin_4); no longer J7.8 (Pin_8)
- net MOSI: now also J7.5 (Pin_5); no longer J7.4 (Pin_4)
- net at J2.1 (A), R6.2, R7.2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: now also Q3.3, R4.1; no longer Q3.2
- net at SW12.2 (B), SW16.2 (B), SW4.1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: now also SW8.2; no longer SW8.1
- net at C18.1, R4.2: now also Q6.3, SW1.2
- new net: D10.1 (K), D11.1 (K), D12.1 (K), D13.1 (K), R27.2, U13.13 (D2)
- new net: D11.2 (A), SW15.1 (A)
- new net: D14.1 (K), D15.1 (K), D16.1 (K), D17.1 (K), R26.2, U13.12 (D1)
- new net: D10.2 (A), SW16.1 (A)
- new net: D12.2 (A), SW14.1
- new net: D6.2 (A), SW8.1
- new net: D13.2 (A), SW9.1
- new net: D20.2 (A), SW6.1
- new net: D21.2 (A), SW17.1
- new net: D6.1 (K), D7.1 (K), D8.1 (K), D9.1 (K), R21.2, U13.14 (D3)
- new net: D8.2 (A), SW18.1
- new net: D16.2 (A), SW10.1
- new net: D14.2 (A), SW12.1 (A)
- new net: D7.2 (A), SW19.1 (A)
- new net: D18.1 (K), D19.1 (K), D20.1 (K), D21.1 (K), R25.2, U13.11 (D0)
- new net: D19.2 (A), SW7.1 (A)
- new net: D17.2 (A), SW13.1
- new net: D18.2 (A), SW4.2
- new net: D9.2 (A), SW5.1
- new net: D15.2 (A), SW11.1 (A)
Other:
- moved on the sheet: BZ1, C18, C20, C23, C27, C28, D4, D5, H1, H2, H3, H4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

Commit message: add pcb interface
Parts:
- added C29: 0.1u, Capacitor_SMD:C_0603_1608Metric_Pad1.08x0.95mm_HandSolder, symbol Device:C_Small
- added D22: WS2812B, LED_SMD:LED_WS2812B_PLCC4_5.0x5.0mm_P3.2mm, symbol LED:WS2812B
- added D24: Green, Diode_SMD:D_1206_3216Metric_Pad1.42x1.75mm_HandSolder, symbol Device:LED_Small
- added R29: 10K, Resistor_SMD:R_0603_1608Metric_Pad0.98x0.95mm_HandSolder, symbol Device:R_Small_US
- added R30: 5.1K, Resistor_SMD:R_0603_1608Metric_Pad0.98x0.95mm_HandSolder, symbol Device:R_Small_US
Connections:
- net +3.3V_Perip: now also C29.2, D22.1 (VDD), R29.2
- net GND: now also C29.1, D22.3 (VSS), D24.1 (K)
- net RGB_LED: now reaches U6.8 (IO15)
- net RGB_LED: now also D22.4 (DIN), R29.1
- net DEFAULT_LED: now reaches U6.9 (IO16)
- net DEFAULT_LED: now also R30.2
- new net: D24.2 (A), R30.1
Other:
- moved on the sheet: C2, C20, C21, C22, C24, C25, C26, C3, D4, D5, JP1, M1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
